Commit message: force xacro to use coarse model

File: yumi_description/urdf/Grippers/yumi_servo_gripper.xacro (robot description, xacro)
@@ -27,5 +27,5 @@
         <origin xyz="0 0 0" rpy="0 0 0"/>
         <geometry>
-          <mesh filename="package://yumi_description/meshes/gripper/base.stl"/>
+          <mesh filename="package://yumi_description/meshes/gripper/coarse/base.stl"/>
         </geometry>
         <material name="Light_Grey"/>
@@ -54,5 +54,5 @@
         <origin xyz="0 0 0" rpy="0 0 0"/>
         <geometry>
-          <mesh filename="package://yumi_description/meshes/gripper/finger.stl"/>
+          <mesh filename="package://yumi_description/meshes/gripper/coarse/finger.stl"/>
         </geometry>
         <material name="Blue"/>
@@ -82,5 +82,5 @@
         <origin xyz="0 0 0" rpy="0 0 0"/>
         <geometry>
-          <mesh filename="package://yumi_description/meshes/gripper/finger.stl"/>
+          <mesh filename="package://yumi_description/meshes/gripper/coarse/finger.stl"/>
         </geometry>
         <material name="Blue"/>

File: yumi_description/urdf/yumi.xacro (robot description, xacro)
@@ -24,5 +24,5 @@
         <origin xyz="0 0 0" rpy="0 0 0"/>
         <geometry>
-          <mesh filename="package://yumi_description/meshes/body.stl"/>
+          <mesh filename="package://yumi_description/meshes/coarse/body.stl"/>
         </geometry>
         <material name="Light_Grey"/>
@@ -56,5 +56,5 @@
         <origin xyz="0 0 0" rpy="0 0 0"/>
         <geometry>
-          <mesh filename="package://yumi_description/meshes/link_1.stl"/>
+          <mesh filename="package://yumi_description/meshes/coarse/link_1.stl"/>
         </geometry>
         <material name="Grey"/>
@@ -87,5 +87,5 @@
         <origin xyz="0 0 0" rpy="0 0 0"/>
         <geometry>
-          <mesh filename="package://yumi_description/meshes/link_2.stl"/>
+          <mesh filename="package://yumi_description/meshes/coarse/link_2.stl"/>
         </geometry>
         <material name="Grey"/>
@@ -118,5 +118,5 @@
         <origin xyz="0 0 0" rpy="0 0 0"/>
         <geometry>
-          <mesh filename="package://yumi_description/meshes/link_3.stl"/>
+          <mesh filename="package://yumi_description/meshes/coarse/link_3.stl"/>
         </geometry>
         <material name="Grey"/>
@@ -149,5 +149,5 @@
         <origin xyz="0 0 0" rpy="0 0 0"/>
         <geometry>
-          <mesh filename="package://yumi_description/meshes/link_4.stl"/>
+          <mesh filename="package://yumi_description/meshes/coarse/link_4.stl"/>
         </geometry>
         <material name="Grey"/>
@@ -180,5 +180,5 @@
         <origin xyz="0 0 0" rpy="0 0 0"/>
         <geometry>
-          <mesh filename="package://yumi_description/meshes/link_5.stl"/>
+          <mesh filename="package://yumi_description/meshes/coarse/link_5.stl"/>
         </geometry>
         <material name="Grey"/>
@@ -211,5 +211,5 @@
         <origin xyz="0 0 0" rpy="0 0 0"/>
         <geometry>
-          <mesh filename="package://yumi_description/meshes/link_6.stl"/>
+          <mesh filename="package://yumi_description/meshes/coarse/link_6.stl"/>
         </geometry>
         <material name="Grey"/>
@@ -242,5 +242,5 @@
         <origin xyz="0 0 0" rpy="0 0 0"/>
         <geometry>
-          <mesh filename="package://yumi_description/meshes/link_7.stl"/>
+          <mesh filename="package://yumi_description/meshes/coarse/link_7.stl"/>
         </geometry>
         <material name="Grey"/>
@@ -274,5 +274,5 @@
         <origin xyz="0 0 0" rpy="0 0 0"/>
         <geometry>
-          <mesh filename="package://yumi_description/meshes/link_1.stl"/>
+          <mesh filename="package://yumi_description/meshes/coarse/link_1.stl"/>
         </geometry>
         <material name="Grey"/>
@@ -305,5 +305,5 @@
         <origin xyz="0 0 0" rpy="0 0 0"/>
         <geometry>
-          <mesh filename="package://yumi_description/meshes/link_2.stl"/>
+          <mesh filename="package://yumi_description/meshes/coarse/link_2.stl"/>
         </geometry>
         <material name="Grey"/>
@@ -336,5 +336,5 @@
         <origin xyz="0 0 0" rpy="0 0 0"/>
         <geometry>
-          <mesh filename="package://yumi_description/meshes/link_3.stl"/>
+          <mesh filename="package://yumi_description/meshes/coarse/link_3.stl"/>
         </geometry>
         <material name="Grey"/>
@@ -367,5 +367,5 @@
         <origin xyz="0 0 0" rpy="0 0 0"/>
         <geometry>
-          <mesh filename="package://yumi_description/meshes/link_4.stl"/>
+          <mesh filename="package://yumi_description/meshes/coarse/link_4.stl"/>
         </geometry>
         <material name="Grey"/>
@@ -398,5 +398,5 @@
         <origin xyz="0 0 0" rpy="0 0 0"/>
         <geometry>
-          <mesh filename="package://yumi_description/meshes/link_5.stl"/>
+          <mesh filename="package://yumi_description/meshes/coarse/link_5.stl"/>
         </geometry>
         <material name="Grey"/>
@@ -429,5 +429,5 @@
         <origin xyz="0 0 0" rpy="0 0 0"/>
         <geometry>
-          <mesh filename="package://yumi_description/meshes/link_6.stl"/>
+          <mesh filename="package://yumi_description/meshes/coarse/link_6.stl"/>
         </geometry>
         <material name="Grey"/>
@@ -460,5 +460,5 @@
         <origin xyz="0 0 0" rpy="0 0 0"/>
         <geometry>
-          <mesh filename="package://yumi_description/meshes/link_7.stl"/>
+          <mesh filename="package://yumi_description/meshes/coarse/link_7.stl"/>
         </geometry>
         <material name="Grey"/>

Commit message: Updated to galactic

File: yumi_description/urdf/Grippers/yumi_servo_gripper.xacro (robot description, xacro)
@@ -5,5 +5,5 @@
     <!-- Import Transmissions -->
     <xacro:include filename="$(find yumi_description)/urdf/Grippers/yumi_servo_gripper.transmission.xacro" />
-    <xacro:include filename="$(find hector_xacro_tools)/urdf/inertia_tensors.urdf.xacro" />
+    <xacro:include filename="$(find yumi_description)/urdf/hector_xacro_tools/inertia_tensors.urdf.xacro" />
     <!-- some constants -->
     <xacro:property name="joint_damping" value="0.5" />

File: yumi_description/urdf/yumi.urdf.xacro (robot description, xacro)
@@ -11,16 +11,5 @@
   <!-- Import Gazebo plugins -->
   <xacro:include filename="$(find yumi_description)/urdf/Gazebo/gazebo.urdf.xacro"/>
-  <!--yumi-->
-  <xacro:yumi name="yumi" hardware_interface="hardware_interface/$(arg arms_interface)" parent="${yumi_parent}" >
-    <origin xyz="0 0 0.1" rpy="0 0 0" />
-  </xacro:yumi>
-  <!--right gripper-->
-  <xacro:yumi_servo_gripper name="gripper_r" hardware_interface="hardware_interface/$(arg grippers_interface)" parent="yumi_link_7_r">
-    <origin xyz="0 0 0.007" rpy="0 0 ${PI}" />
-  </xacro:yumi_servo_gripper>
-  <!--left gripper-->
-  <xacro:yumi_servo_gripper name="gripper_l" hardware_interface="hardware_interface/$(arg grippers_interface)" parent="yumi_link_7_l">
-    <origin xyz="0 0 0.007" rpy="0 0 ${PI}" />
-  </xacro:yumi_servo_gripper>
+  <!-- Yumi Setup -->
   <xacro:property name="yumi_setup" value="$(arg yumi_setup)" />
   <xacro:if value="${yumi_setup == 'robot_centric'}">
@@ -36,3 +25,15 @@
     </joint>
   </xacro:if>
+  <!--yumi-->
+  <xacro:yumi name="yumi" hardware_interface="hardware_interface/$(arg arms_interface)" parent="${yumi_parent}" >
+    <origin xyz="0 0 0.1" rpy="0 0 0" />
+  </xacro:yumi>
+  <!--right gripper-->
+  <xacro:yumi_servo_gripper name="gripper_r" hardware_interface="hardware_interface/$(arg grippers_interface)" parent="yumi_link_7_r">
+    <origin xyz="0 0 0.007" rpy="0 0 ${PI}" />
+  </xacro:yumi_servo_gripper>
+  <!--left gripper-->
+  <xacro:yumi_servo_gripper name="gripper_l" hardware_interface="hardware_interface/$(arg grippers_interface)" parent="yumi_link_7_l">
+    <origin xyz="0 0 0.007" rpy="0 0 ${PI}" />
+  </xacro:yumi_servo_gripper>
 </robot>

Commit message: Simple visualization of Yumi in Rviz, controlled with jsp gui

File: yumi_description/urdf/Grippers/yumi_servo_gripper.xacro (robot description, xacro)
@@ -5,5 +5,5 @@
     <!-- Import Transmissions -->
     <xacro:include filename="$(find yumi_description)/urdf/Grippers/yumi_servo_gripper.transmission.xacro" />
-    <xacro:include filename="$(find hector_xacro_tools)/urdf/inertia_tensors.urdf.xacro" />
+    <!--<xacro:include filename="$(find hector_xacro_tools)/urdf/inertia_tensors.urdf.xacro" />-->
     <!-- some constants -->
     <xacro:property name="joint_damping" value="0.5" />
@@ -50,5 +50,5 @@
     </joint>
     <link name="${name}_finger_r">
-      <xacro:inertial_cuboid mass="0.04" x_length="0.05" y_length="0.05" z_length="0.05" />
+      <!--<xacro:inertial_cuboid mass="0.04" x_length="0.05" y_length="0.05" z_length="0.05" />--> <!-- hector_xacro_tools not in ROS2 -->
       <visual>
         <origin xyz="0 0 0" rpy="0 0 0"/>
@@ -78,5 +78,5 @@
     </joint>
     <link name="${name}_finger_l">
-      <xacro:inertial_cuboid mass="0.04" x_length="0.05" y_length="0.05" z_length="0.05" />
+      <!--<xacro:inertial_cuboid mass="0.04" x_length="0.05" y_length="0.05" z_length="0.05" />--> <!-- hector_xacro_tools not in ROS2 -->
       <visual>
         <origin xyz="0 0 0" rpy="0 0 0"/>

File: yumi_description/urdf/yumi.urdf.xacro (robot description, xacro)
@@ -11,16 +11,4 @@
   <!-- Import Gazebo plugins -->
   <xacro:include filename="$(find yumi_description)/urdf/Gazebo/gazebo.urdf.xacro"/>
-  <!--yumi-->
-  <xacro:yumi name="yumi" hardware_interface="hardware_interface/$(arg arms_interface)" parent="${yumi_parent}" >
-    <origin xyz="0 0 0.1" rpy="0 0 0" />
-  </xacro:yumi>
-  <!--right gripper-->
-  <xacro:yumi_servo_gripper name="gripper_r" hardware_interface="hardware_interface/$(arg grippers_interface)" parent="yumi_link_7_r">
-    <origin xyz="0 0 0.007" rpy="0 0 ${PI}" />
-  </xacro:yumi_servo_gripper>
-  <!--left gripper-->
-  <xacro:yumi_servo_gripper name="gripper_l" hardware_interface="hardware_interface/$(arg grippers_interface)" parent="yumi_link_7_l">
-    <origin xyz="0 0 0.007" rpy="0 0 ${PI}" />
-  </xacro:yumi_servo_gripper>
   <xacro:property name="yumi_setup" value="$(arg yumi_setup)" />
   <xacro:if value="${yumi_setup == 'robot_centric'}">
@@ -36,3 +24,15 @@
     </joint>
   </xacro:if>
+  <!--yumi-->
+  <xacro:yumi name="yumi" hardware_interface="hardware_interface/$(arg arms_interface)" parent="${yumi_parent}" >
+    <origin xyz="0 0 0.1" rpy="0 0 0" />
+  </xacro:yumi>
+  <!--right gripper-->
+  <xacro:yumi_servo_gripper name="gripper_r" hardware_interface="hardware_interface/$(arg grippers_interface)" parent="yumi_link_7_r">
+    <origin xyz="0 0 0.007" rpy="0 0 ${PI}" />
+  </xacro:yumi_servo_gripper>
+  <!--left gripper-->
+  <xacro:yumi_servo_gripper name="gripper_l" hardware_interface="hardware_interface/$(arg grippers_interface)" parent="yumi_link_7_l">
+    <origin xyz="0 0 0.007" rpy="0 0 ${PI}" />
+  </xacro:yumi_servo_gripper>
 </robot>
