Commit message: Compiles and seems to work in Gazebo/Rviz in 20.04

File: yumi_description/urdf/yumi.urdf.xacro (robot description, xacro)
@@ -11,4 +11,5 @@
   <!-- Import Gazebo plugins -->
   <xacro:include filename="$(find yumi_description)/urdf/Gazebo/gazebo.urdf.xacro"/>
+  <xacro:property name="yumi_parent" default="world"/>
   <!--yumi-->
   <xacro:yumi name="yumi" hardware_interface="hardware_interface/$(arg arms_interface)" parent="${yumi_parent}" >

Commit message: Updated yumi to not use world as base link, that messes up with RDFModel. bug

File: yumi_description/urdf/yumi.urdf.xacro (robot description, xacro)
@@ -25,5 +25,6 @@
   </xacro:if>
   <!--yumi-->
-  <xacro:yumi name="yumi" hardware_interface="hardware_interface/$(arg arms_interface)" parent="${yumi_parent}" >
+  <!--<xacro:yumi name="yumi" hardware_interface="hardware_interface/$(arg arms_interface)" parent="${yumi_parent}" > -->
+  <xacro:yumi name="yumi" hardware_interface="hardware_interface/$(arg arms_interface)">
     <origin xyz="0 0 0.1" rpy="0 0 0" />
   </xacro:yumi>

File: yumi_description/urdf/yumi.xacro (robot description, xacro)
@@ -8,5 +8,5 @@
   <xacro:property name="joint_damping" value="0.5" />
   <xacro:property name="max_effort" value="300"/>
-  <xacro:macro name="yumi" params="parent name hardware_interface *origin">
+  <xacro:macro name="yumi" params="name hardware_interface *origin">
     <link name="yumi_base_link"></link>
     <joint name="${name}_base_link_to_body" type="fixed">

Commit message: Actually use the xyz and rpy arguments

File: yumi_description/urdf/yumi.urdf.xacro (robot description, xacro)
@@ -21,5 +21,5 @@
       <parent link="world"/>
       <child link="yumi_base_link"/>
-      <origin xyz="0 0 0.1" rpy="0 0 0" />
+      <origin xyz="$(arg xyz)" rpy="$(arg rpy)" />
     </joint>
   </xacro:if>
